File: Project 4 MCU Datalogger.kicad_pcb (KiCad board)
At the start: 2 copper layers, 48.5 x 33.3 mm, 30 parts, among them J1 Conn_02x03_Odd_Even, J2 Conn_01x04_Pin, J3 Conn_01x09_Pin, J4 Conn_01x04_Pin, U1 24LC1025, U2 24LC1025, U3 DS1337S_, U4 ATMEGA328P-AU, Y1 32.768kHZ, Y2 16MHz

Commit message: Completed 2-layer Pcb project.
Routing:
- net /Vcc: track 142.4 -> 173.6 mm, vias 23 -> 20
Other:
- board text added: "0.0000 mm / 0.0000 mm"
- board text added: "0.3000 mm"
- board text added: "1.6000 mm"
- board text added: "48.5212 mm x 33.2812 mm"
- board text added: "BOARD CHARACTERISTICS"
- board text added: "Board Thickness:"
- board text added: "Board overall dimensions:"
- board text added: "Castellated pads:"
- board text added: "Copper Finish:"
- board text added: "Copper Layer Count:"
- board text added: "Edge card connectors:"
- board text added: "Impedance Control:"
- board text added: "Min hole diameter:"
- board text added: "Min track/spacing:"
- board text added: "No"
- board text added: "None"
- board text added: "Plated Board Edge:"
