File: Project 4 MCU Datalogger.kicad_pcb (KiCad board)
At the start: 4 copper layers, 48.5 x 33.3 mm, 30 parts, among them J1 Conn_02x03_Odd_Even, J2 Conn_01x04_Pin, J3 Conn_01x09_Pin, J4 Conn_01x04_Pin, U1 24LC1025, U2 24LC1025, U3 DS1337S_, U4 ATMEGA328P-AU, Y1 32.768kHZ, Y2 16MHz

Commit message: Added extra tracks.
Routing:
- net GND: track 54.6 -> 54.0 mm
Changed lines of the file:
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@@
-	)
-	(segment
-		(start 114.554 84.836)
-		(end 114.046 85.344)
-		(width 0.35)
-		(layer "B.Cu")
-		(net 2)
 	)
 	(segment
@@
 	)
 	(segment
-		(start 114.046 85.344)
+		(start 114.046 86.36)
 		(end 114.046 88.2396)
 		(width 0.35)
@@
 	(segment
 		(start 116.9924 84.836)
-		(end 114.554 84.836)
+		(end 115.57 84.836)
+		(width 0.35)
+		(layer "B.Cu")
+		(net 2)
+	)
+	(segment
+		(start 114.046 86.36)
+		(end 115.57 84.836)
 		(width 0.35)
 		(layer "B.Cu")
@@
 	)
 	(segment
+		(start 143.51 83.185)
+		(end 145.0594 83.185)
+		(width 0.25)
+		(layer "F.Cu")
+		(net 9)
+	)
+	(segment
 		(start 134.3616 93.07)
 		(end 134.4168 93.0148)
@@
 	)
 	(segment
-		(start 145.0086 83.185)
-		(end 143.51 83.185)
+		(start 145.4912 83.6168)
+		(end 145.4912 84.4296)
 		(width 0.25)
 		(layer "F.Cu")
@@
 	)
 	(segment
-		(start 145.4912 83.6168)
-		(end 145.034 83.1596)
-		(width 0.25)
-		(layer "F.Cu")
-		(net 9)
-	)
-	(segment
-		(start 145.4912 84.4296)
+		(start 145.0594 83.185)
 		(end 145.4912 83.6168)
 		(width 0.25)
 		(layer "F.Cu")
-		(net 9)
-	)
-	(segment
-		(start 145.034 83.1596)
-		(end 145.0086 83.185)
-		(width 0.25)
-		(layer "F.Cu")
